Commit message: feat: add sensor kit change for simulation

File: aichallenge/workspace/src/aichallenge_submit/racing_kart_sensor_kit_description/urdf/sensor_kit.xacro (robot description, xacro)
@@ -5,4 +5,5 @@
     <xacro:arg name="gpu" default="false"/>
     <xacro:arg name="config_dir" default="$(find racing_kart_sensor_kit_description)/config"/>
+    <xacro:arg name="simulation" default="false"/>
     <xacro:property name="sensor_kit_base_link" default="sensor_kit_base_link"/>
     <joint name="${sensor_kit_base_link}_joint" type="fixed">
@@ -16,4 +17,8 @@
     <!-- sensor -->
     <xacro:property name="calibration" value="${xacro.load_yaml('$(arg config_dir)/sensor_kit_calibration.yaml')}"/>
+    <!-- over write calibration file for simulation -->
+    <xacro:if value="$(arg simulation)">
+      <xacro:property name="calibration" value="${xacro.load_yaml('$(arg config_dir)/awsim_sensor_kit_calibration.yaml')}"/>
+    </xacro:if>
     <!-- gnss -->
     <xacro:imu_macro
