Commit message: add racing kart model

File: aichallenge/workspace/src/aichallenge_submit/racing_kart_description/urdf/vehicle.xacro (robot description, xacro)
@@ -6,7 +6,7 @@
   <link name="base_link">
     <visual>
-      <origin xyz="0 0 0" rpy="0 0 0"/>
+      <origin xyz="0 0 0" rpy="0 0 1.57"/>
       <geometry>
-        <mesh filename="package://racing_kart_description/mesh/square.dae" scale="1 1 1"/>
+        <mesh filename="package://racing_kart_description/mesh/kart.dae" scale="1 1 1"/>
       </geometry>
     </visual>
